File: Hardware/SparkX-Pi-Filter.sch (EAGLE design)
At the start: 14 parts

Commit message: Added Screw Terminals and adjusted labels
Added Screw Terminals and adjusted labels
Parts:
- removed J3, J4: (no value), SparkFun-Connectors:CONN_01PTH_NO_SILK_YES_STOP
- J1, J2: device SparkFun-Connectors:CONN_01PTH_NO_SILK_YES_STOP -> SparkFun-Connectors:CONN_022.54MM_SCREWTERM
Connections:
- net GND: now also J1.2; no longer J4.1
- net N$2: now also J2.2; no longer J3.1
Changed lines of the file:
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@@
 <part name="GND1" library="SparkFun-PowerSymbols" deviceset="GND" device=""/>
 <part name="GND2" library="SparkFun-PowerSymbols" deviceset="GND" device=""/>
-<part name="J1" library="SparkFun-Connectors" deviceset="CONN_01" device="PTH_NO_SILK_YES_STOP"/>
-<part name="J2" library="SparkFun-Connectors" deviceset="CONN_01" device="PTH_NO_SILK_YES_STOP"/>
-<part name="J3" library="SparkFun-Connectors" deviceset="CONN_01" device="PTH_NO_SILK_YES_STOP"/>
-<part name="J4" library="SparkFun-Connectors" deviceset="CONN_01" device="PTH_NO_SILK_YES_STOP"/>
 <part name="H1" library="SparkFun-Hardware" deviceset="STAND-OFF" device=""/>
 <part name="H2" library="SparkFun-Hardware" deviceset="STAND-OFF" device=""/>
@@
 <part name="U$1" library="SparkX" deviceset="SPARKX-LOGO" device="4"/>
 <part name="LOGO1" library="SparkFun-Aesthetics" deviceset="OSHW-LOGO" device="M"/>
+<part name="J1" library="SparkFun-Connectors" deviceset="CONN_02" device="2.54MM_SCREWTERM"/>
+<part name="J2" library="SparkFun-Connectors" deviceset="CONN_02" device="2.54MM_SCREWTERM"/>
 </parts>
 <sheets>
@@
 <attribute name="VALUE" x="134.62" y="88.646" size="1.778" layer="96" align="top-center"/>
 </instance>
-<instance part="J1" gate="G$1" x="91.44" y="109.22" smashed="yes">
-<attribute name="VALUE" x="88.9" y="104.394" size="1.778" layer="96" font="vector"/>
-<attribute name="NAME" x="88.9" y="112.268" size="1.778" layer="95" font="vector"/>
-</instance>
-<instance part="J2" gate="G$1" x="91.44" y="93.98" smashed="yes">
-<attribute name="VALUE" x="88.9" y="89.154" size="1.778" layer="96" font="vector"/>
-<attribute name="NAME" x="88.9" y="97.028" size="1.778" layer="95" font="vector"/>
-</instance>
-<instance part="J3" gate="G$1" x="154.94" y="109.22" smashed="yes" rot="MR0">
-<attribute name="VALUE" x="157.48" y="104.394" size="1.778" layer="96" font="vector" rot="MR0"/>
-<attribute name="NAME" x="157.48" y="112.268" size="1.778" layer="95" font="vector" rot="MR0"/>
-</instance>
-<instance part="J4" gate="G$1" x="154.94" y="93.98" smashed="yes" rot="MR0">
-<attribute name="VALUE" x="157.48" y="89.154" size="1.778" layer="96" font="vector" rot="MR0"/>
-<attribute name="NAME" x="157.48" y="97.028" size="1.778" layer="95" font="vector" rot="MR0"/>
-</instance>
 <instance part="H1" gate="G$1" x="246.38" y="25.4" smashed="yes"/>
 <instance part="H2" gate="G$1" x="246.38" y="30.48" smashed="yes"/>
@@
 <instance part="U$1" gate="G$1" x="15.24" y="177.8" smashed="yes"/>
 <instance part="LOGO1" gate="G$1" x="236.22" y="177.8" smashed="yes"/>
+<instance part="J1" gate="G$1" x="88.9" y="104.14" smashed="yes" rot="MR180">
+<attribute name="VALUE" x="86.36" y="108.966" size="1.778" layer="96" font="vector" rot="MR180"/>
+<attribute name="NAME" x="86.36" y="98.552" size="1.778" layer="95" font="vector" rot="MR180"/>
+</instance>
+<instance part="J2" gate="G$1" x="157.48" y="101.6" smashed="yes" rot="MR0">
+<attribute name="VALUE" x="160.02" y="96.774" size="1.778" layer="96" font="vector" rot="MR0"/>
+<attribute name="NAME" x="160.02" y="107.188" size="1.778" layer="95" font="vector" rot="MR0"/>
+</instance>
 </instances>
 <busses>
@@
 <wire x1="111.76" y1="109.22" x2="99.06" y2="109.22" width="0.1524" layer="91"/>
 <junction x="111.76" y="109.22"/>
+<wire x1="99.06" y1="109.22" x2="99.06" y2="104.14" width="0.1524" layer="91"/>
 <pinref part="J1" gate="G$1" pin="1"/>
+<wire x1="99.06" y1="104.14" x2="96.52" y2="104.14" width="0.1524" layer="91"/>
 </segment>
 </net>
@@
 <wire x1="134.62" y1="109.22" x2="147.32" y2="109.22" width="0.1524" layer="91"/>
 <junction x="134.62" y="109.22"/>
-<pinref part="J3" gate="G$1" pin="1"/>
+<wire x1="147.32" y1="109.22" x2="147.32" y2="104.14" width="0.1524" layer="91"/>
+<pinref part="J2" gate="G$1" pin="2"/>
+<wire x1="147.32" y1="104.14" x2="149.86" y2="104.14" width="0.1524" layer="91"/>
 </segment>
 </net>
@@
 <wire x1="111.76" y1="93.98" x2="99.06" y2="93.98" width="0.1524" layer="91"/>
 <junction x="111.76" y="93.98"/>
-<pinref part="J2" gate="G$1" pin="1"/>
+<pinref part="J1" gate="G$1" pin="2"/>
+<wire x1="99.06" y1="93.98" x2="99.06" y2="101.6" width="0.1524" layer="91"/>
+<wire x1="99.06" y1="101.6" x2="96.52" y2="101.6" width="0.1524" layer="91"/>
 </segment>
 <segment>
@@
 <wire x1="134.62" y1="93.98" x2="147.32" y2="93.98" width="0.1524" layer="91"/>
 <junction x="134.62" y="93.98"/>
-<pinref part="J4" gate="G$1" pin="1"/>
+<wire x1="147.32" y1="93.98" x2="147.32" y2="101.6" width="0.1524" layer="91"/>
+<pinref part="J2" gate="G$1" pin="1"/>
+<wire x1="149.86" y1="101.6" x2="147.32" y2="101.6" width="0.1524" layer="91"/>
 </segment>
 </net>
